File: PCB/Macro pad copy.kicad_pcb (KiCad board)
At the start: 2 copper layers, 58.5 x 96 mm, 6 parts, among them SW1 SW_Push, SW2 SW_Push, SW3 SW_Push, SW4 SW_Push, U1 ER_OLEDM0.91_1x-I2C, U2 MOUDLE-SEEEDUINO-XIAO

Commit message: Add files via upload
Parts:
- added G***: LOGO, IMages:logo, F.Cu at (148.0, 105.5)
Routing:
- net Net-(U2-PA10_A2_D2): track 92.2 -> 94.4 mm
- net GND: track 148.1 -> 150.3 mm
- net Net-(U2-PA7_A8_D8_SCK): track 24.6 -> 25.2 mm
